File: Orion.kicad_pcb (KiCad board)
At the start: 2 copper layers, 60 x 60 mm, 27 parts, among them J1 USB_A, J2 USB_A, J3 USB_A, J4 USB_A, U1 FE1.1s, U2 PRTR5V0U2X, Y1 12MHz

Commit message: Add render
Parts:
- added U3: PRTR5V0U2X, random-keyboard-parts:SOT143B, F.Cu at (96.0, 60.0)
- added U4: PRTR5V0U2X, random-keyboard-parts:SOT143B, F.Cu at (64.0, 81.0)
- added U5: PRTR5V0U2X, random-keyboard-parts:SOT143B, F.Cu at (96.0, 81.0)
- added U6: PRTR5V0U2X, random-keyboard-parts:SOT143B, F.Cu at (64.0, 59.0)
Routing:
- net GNDA: track 176.7 -> 218.9 mm
- net GND: track 362.8 -> 369.7 mm
- net Net-(F2-Pad2): track 4.12 -> 7.32 mm
- net Net-(F4-Pad2): track 4.12 -> 7.32 mm
- net Net-(F3-Pad2): track 4.12 -> 7.32 mm
- net Net-(F1-Pad2): track 4.12 -> 7.32 mm
- net D4-: track 41.1 -> 43.4 mm
- net D4+: track 41.7 -> 43.5 mm
- net D1+: track 37.9 -> 39.3 mm
- net D1-: track 38.4 -> 39.5 mm
- net D3+: track 32.9 -> 33.6 mm
- net D2+: track 32.3 -> 33.0 mm
- net D3-: track 32.3 -> 33.0 mm
- net D2-: track 32.9 -> 33.6 mm
Other:
- net class Power: trace_width 0.635 -> 0.508
